File: CANBoard-Base/AnalogInputs.kicad_sch (KiCad schematic)
At the start: 46 parts, among them U2 LM324, U3 LM324, U4 SRV05-4, U5 SRV05-4

Commit message: change to mcp6004
Parts:
- U2, U3: value LM324 -> MCP6004; symbol Amplifier_Operational:LM324 -> Amplifier_Operational:MCP6004; JLC_PN C7942 -> C50282
Changed lines of the file:
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@@
 	)
 	(symbol
-		(lib_id "Amplifier_Operational:LM324")
+		(lib_id "Amplifier_Operational:MCP6004")
 		(at 245.11 27.94 0)
 		(unit 5)
@@
 		(fields_autoplaced yes)
 		(property "Reference" "U3"
-			(at 243.205 26.7279 0)
+			(at 243.205 26.7278 0)
 			(effects
 				(font
@@
 			)
 		)
-		(property "Value" "LM324"
+		(property "Value" "MCP6004"
 			(at 243.205 29.1521 0)
 			(effects
@@
 			)
 		)
-		(property "Datasheet" "http://www.ti.com/lit/ds/symlink/lm2902-n.pdf"
+		(property "Datasheet" "http://ww1.microchip.com/downloads/en/DeviceDoc/21733j.pdf"
 			(at 246.38 22.86 0)
 			(effects
@@
 			)
 		)
-		(property "Description" ""
+		(property "Description" "1MHz, Low-Power Op Amp, DIP-14/SOIC-14/TSSOP-14"
 			(at 245.11 27.94 0)
 			(effects
@@
 			)
 		)
-		(property "JLC_PN" "C7942"
+		(property "JLC_PN" "C50282"
 			(at 245.11 27.94 0)
 			(effects
@@
 	)
 	(symbol
-		(lib_id "Amplifier_Operational:LM324")
+		(lib_id "Amplifier_Operational:MCP6004")
 		(at 191.77 93.98 0)
 		(unit 1)
@@
 		(fields_autoplaced yes)
 		(property "Reference" "U2"
-			(at 191.77 84.7557 0)
+			(at 191.77 84.7555 0)
 			(effects
 				(font
@@
 			)
 		)
-		(property "Value" "LM324"
-			(at 191.77 87.1799 0)
+		(property "Value" "MCP6004"
+			(at 191.77 87.1798 0)
 			(effects
 				(font
@@
 			)
 		)
-		(property "Datasheet" "http://www.ti.com/lit/ds/symlink/lm2902-n.pdf"
+		(property "Datasheet" "http://ww1.microchip.com/downloads/en/DeviceDoc/21733j.pdf"
 			(at 193.04 88.9 0)
 			(effects
@@
 			)
 		)
-		(property "Description" ""
+		(property "Description" "1MHz, Low-Power Op Amp, DIP-14/SOIC-14/TSSOP-14"
 			(at 191.77 93.98 0)
 			(effects
@@
 			)
 		)
-		(property "JLC_PN" "C7942"
+		(property "JLC_PN" "C50282"
 			(at 191.77 93.98 0)
 			(effects
@@
 	)
 	(symbol
-		(lib_id "Amplifier_Operational:LM324")
+		(lib_id "Amplifier_Operational:MCP6004")
 		(at 191.77 74.93 0)
 		(unit 3)
@@
 		(fields_autoplaced yes)
 		(property "Reference" "U2"
-			(at 191.77 65.7057 0)
+			(at 191.77 65.7055 0)
 			(effects
 				(font
@@
 			)
 		)
-		(property "Value" "LM324"
-			(at 191.77 68.1299 0)
+		(property "Value" "MCP6004"
+			(at 191.77 68.1298 0)
 			(effects
 				(font
@@
 			)
 		)
-		(property "Datasheet" "http://www.ti.com/lit/ds/symlink/lm2902-n.pdf"
+		(property "Datasheet" "http://ww1.microchip.com/downloads/en/DeviceDoc/21733j.pdf"
 			(at 193.04 69.85 0)
 			(effects
@@
 			)
 		)
-		(property "Description" ""
+		(property "Description" "1MHz, Low-Power Op Amp, DIP-14/SOIC-14/TSSOP-14"
 			(at 191.77 74.93 0)
 			(effects
@@
 			)
 		)
-		(property "JLC_PN" "C7942"
+		(property "JLC_PN" "C50282"
 			(at 191.77 74.93 0)
 			(effects
@@
 	)
 	(symbol
-		(lib_id "Amplifier_Operational:LM324")
+		(lib_id "Amplifier_Operational:MCP6004")
 		(at 215.9 27.94 0)
 		(unit 5)
@@
 		(fields_autoplaced yes)
 		(property "Reference" "U2"
-			(at 213.995 26.7279 0)
+			(at 213.995 26.7278 0)
 			(effects
 				(font
@@
 			)
 		)
-		(property "Value" "LM324"
+		(property "Value" "MCP6004"
 			(at 213.995 29.1521 0)
 			(effects
@@
 			)
 		)
-		(property "Datasheet" "http://www.ti.com/lit/ds/symlink/lm2902-n.pdf"
+		(property "Datasheet" "http://ww1.microchip.com/downloads/en/DeviceDoc/21733j.pdf"
 			(at 217.17 22.86 0)
 			(effects
@@
 			)
 		)
-		(property "Description" ""
+		(property "Description" "1MHz, Low-Power Op Amp, DIP-14/SOIC-14/TSSOP-14"
 			(at 215.9 27.94 0)
 			(effects
@@
 			)
 		)
-		(property "JLC_PN" "C7942"
+		(property "JLC_PN" "C50282"
 			(at 215.9 27.94 0)
 			(effects
@@
 	)
 	(symbol
-		(lib_id "Amplifier_Operational:LM324")
+		(lib_id "Amplifier_Operational:MCP6004")
 		(at 191.77 55.88 0)
 		(unit 2)
@@
 		(fields_autoplaced yes)
 		(property "Reference" "U2"
-			(at 191.77 46.6557 0)
+			(at 191.77 46.6555 0)
 			(effects
 				(font
@@
 			)
 		)
-		(property "Value" "LM324"
-			(at 191.77 49.0799 0)
+		(property "Value" "MCP6004"
+			(at 191.77 49.0798 0)
 			(effects
 				(font
@@
 			)
 		)
-		(property "Datasheet" "http://www.ti.com/lit/ds/symlink/lm2902-n.pdf"
+		(property "Datasheet" "http://ww1.microchip.com/downloads/en/DeviceDoc/21733j.pdf"
 			(at 193.04 50.8 0)
 			(effects
@@
 			)
 		)
-		(property "Description" ""
+		(property "Description" "1MHz, Low-Power Op Amp, DIP-14/SOIC-14/TSSOP-14"
 			(at 191.77 55.88 0)
 			(effects
@@
 			)
 		)
-		(property "JLC_PN" "C7942"
+		(property "JLC_PN" "C50282"
 			(at 191.77 55.88 0)
 			(effects
@@
 	)
 	(symbol
-		(lib_id "Amplifier_Operational:LM324")
+		(lib_id "Amplifier_Operational:MCP6004")
 		(at 191.77 111.76 0)
 		(unit 3)
@@
 		(fields_autoplaced yes)
 		(property "Reference" "U3"
-			(at 191.77 102.5357 0)
+			(at 191.77 102.5355 0)
 			(effects
 				(font
@@
 			)
 		)
-		(property "Value" "LM324"
-			(at 191.77 104.9599 0)
+		(property "Value" "MCP6004"
+			(at 191.77 104.9598 0)
 			(effects
 				(font
@@
 			)
 		)
-		(property "Datasheet" "http://www.ti.com/lit/ds/symlink/lm2902-n.pdf"
+		(property "Datasheet" "http://ww1.microchip.com/downloads/en/DeviceDoc/21733j.pdf"
 			(at 193.04 106.68 0)
 			(effects
@@
 			)
 		)
-		(property "Description" ""
+		(property "Description" "1MHz, Low-Power Op Amp, DIP-14/SOIC-14/TSSOP-14"
 			(at 191.77 111.76 0)
 			(effects
@@
 			)
 		)
-		(property "JLC_PN" "C7942"
+		(property "JLC_PN" "C50282"
 			(at 191.77 111.76 0)
 			(effects
@@
 	)
 	(symbol
-		(lib_id "Amplifier_Operational:LM324")
+		(lib_id "Amplifier_Operational:MCP6004")
 		(at 191.77 130.81 0)
 		(unit 4)
@@
 		(fields_autoplaced yes)
 		(property "Reference" "U3"
-			(at 191.77 121.5857 0)
+			(at 191.77 121.5855 0)
 			(effects
 				(font
@@
 			)
 		)
-		(property "Value" "LM324"
-			(at 191.77 124.0099 0)
+		(property "Value" "MCP6004"
+			(at 191.77 124.0098 0)
 			(effects
 				(font
@@
 			)
 		)
-		(property "Datasheet" "http://www.ti.com/lit/ds/symlink/lm2902-n.pdf"
+		(property "Datasheet" "http://ww1.microchip.com/downloads/en/DeviceDoc/21733j.pdf"
 			(at 193.04 125.73 0)
 			(effects
@@
 			)
 		)
-		(property "Description" ""
+		(property "Description" "1MHz, Low-Power Op Amp, DIP-14/SOIC-14/TSSOP-14"
 			(at 191.77 130.81 0)
 			(effects
@@
 			)
 		)
-		(property "JLC_PN" "C7942"
+		(property "JLC_PN" "C50282"
 			(at 191.77 130.81 0)
 			(effects
